File: Titan.kicad_pcb (KiCad board)
At the start: 2 copper layers, 285.4 x 94.9 mm, 1 part, among them U1 Outline

Commit message: Add silk, update gerbers
Parts:
- added G***: LOGO, locallib:AI03-Silkscreen-5.4mm, B.Cu at (246.4, 95.0)
- added REF**: ai03-20mil, locallib:ai03-20mil, F.Cu at (124.6, 108.7)
Other:
- board text added: "For default non-ISO layout, optional split back"
- board text added: "Titan - Cut-PCB keyboard plate for Voyager"
- board text added: "www.ai03.me"
Changed lines of the file:
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@@
 (kicad_pcb (version 4) (host pcbnew 4.0.6)
   (general
-    (links 1)
+    (links 0)
     (no_connects 1)
     (area 23.8125 23.8125 317.500001 127.000001)
     (thickness 1.6)
-    (drawings 0)
+    (drawings 4)
     (tracks 0)
     (zones 0)
-    (modules 1)
+    (modules 3)
     (nets 2)
   )
@@
     (pad_to_mask_clearance 0.2)
     (aux_axis_origin 0 0)
-    (visible_elements FFFFFF7F)
+    (visible_elements 7FFFFFFF)
     (pcbplotparams
       (layerselection 0x010f0_80000001)
@@
       (net 1 GND))
   )
+  (module locallib:ai03-20mil (layer F.Cu)
+    (at 124.61875 108.74375)
+    (fp_text reference REF** (at 0 5.08) (layer Dwgs.User)
+      (effects (font (size 1 1) (thickness 0.15)))
+    )
+    (fp_text value ai03-20mil (at 0 -5.08) (layer Dwgs.User)
+      (effects (font (size 1 1) (thickness 0.15)))
+    )
+    (pad 4 smd rect (at -0.508 -0.508) (size 0.508 0.508) (layers F.Cu F.Paste F.Mask))
+    (pad 5 smd rect (at -1.016 0.508) (size 0.508 0.508) (layers F.Cu F.Paste F.Mask))
+    (pad 6 smd rect (at 0 0.508) (size 0.508 0.508) (layers F.Cu F.Paste F.Mask))
+    (pad 7 smd rect (at 1.016 0.508) (size 0.508 0.508) (layers F.Cu F.Paste F.Mask))
+    (pad 8 smd rect (at 0.508 -0.508) (size 0.508 0.508) (layers F.Cu F.Paste F.Mask))
+    (pad 9 smd rect (at 0 -1.524) (size 0.508 0.508) (layers F.Cu F.Paste F.Mask))
+    (pad 10 smd rect (at -1.524 1.524) (size 0.508 0.508) (layers F.Cu F.Paste F.Mask))
+    (pad 11 smd rect (at 1.524 1.524) (size 0.508 0.508) (layers F.Cu F.Paste F.Mask))
+  )
+  (module locallib:AI03-Silkscreen-5.4mm (layer B.Cu)
+    (at 246.38 94.996 180)
+    (fp_text reference G*** (at 0 0 180) (layer B.SilkS) hide
+      (effects (font (thickness 0.3)) (justify mirror))
+    )
+    (fp_text value LOGO (at 0.75 0 180) (layer B.SilkS) hide
+      (effects (font (thickness 0.3)) (justify mirror))
+    )
+    (fp_poly (pts (xy 0.102617 2.717503) (xy 0.181585 2.7149) (xy 0.25454 2.710978) (xy 0.318558 2.705752)
+      (xy 0.359229 2.700946) (xy 0.559507 2.665802) (xy 0.753969 2.617444) (xy 0.942353 2.556002)
+      (xy 1.124401 2.481605) (xy 1.299853 2.394382) (xy 1.468447 2.294464) (xy 1.629926 2.18198)
+      (xy 1.784028 2.057059) (xy 1.930494 1.919831) (xy 1.935528 1.914757) (xy 2.071735 1.767115)
+      (xy 2.195425 1.612181) (xy 2.306484 1.450206) (xy 2.404798 1.281438) (xy 2.490251 1.106128)
+      (xy 2.56273 0.924525) (xy 2.62212 0.736878) (xy 2.668305 0.543437) (xy 2.701173 0.34445)
+      (xy 2.714848 0.217985) (xy 2.718554 0.158194) (xy 2.720496 0.087595) (xy 2.720766 0.009779)
+      (xy 2.719454 -0.071667) (xy 2.716652 -0.153154) (xy 2.712451 -0.231093) (xy 2.706941 -0.301897)
+      (xy 2.700215 -0.361976) (xy 2.700094 -0.362857) (xy 2.665688 -0.561345) (xy 2.617836 -0.754451)
+      (xy 2.556694 -0.941874) (xy 2.482412 -1.12331) (xy 2.395144 -1.298457) (xy 2.295041 -1.467013)
+      (xy 2.182258 -1.628675) (xy 2.056945 -1.783141) (xy 1.919257 -1.930108) (xy 1.900424 -1.948678)
+      (xy 1.752544 -2.083657) (xy 1.598359 -2.205679) (xy 1.437679 -2.314838) (xy 1.270312 -2.411225)
+      (xy 1.096069 -2.494932) (xy 0.914758 -2.566049) (xy 0.72619 -2.62467) (xy 0.530172 -2.670886)
+      (xy 0.3302 -2.704294) (xy 0.302819 -2.707019) (xy 0.263477 -2.709611) (xy 0.214727 -2.712009)
+      (xy 0.159123 -2.714156) (xy 0.099217 -2.715993) (xy 0.037562 -2.717461) (xy -0.023287 -2.718502)
+      (xy -0.080778 -2.719058) (xy -0.132358 -2.71907) (xy -0.175474 -2.718479) (xy -0.207573 -2.717228)
+      (xy -0.214086 -2.716763) (xy -0.412671 -2.693282) (xy -0.607608 -2.65582) (xy -0.798465 -2.60455)
+      (xy -0.984809 -2.539646) (xy -1.166206 -2.46128) (xy -1.342225 -2.369626) (xy -1.512433 -2.264857)
+      (xy -1.676396 -2.147146) (xy -1.715976 -2.116024) (xy -1.761667 -2.077625) (xy -1.813845 -2.030711)
+      (xy -1.869777 -1.977974) (xy -1.926729 -1.922109) (xy -1.981969 -1.865808) (xy -2.032763 -1.811766)
+      (xy -2.076378 -1.762675) (xy -2.085524 -1.751869) (xy -2.208767 -1.593846) (xy -2.31879 -1.430097)
+      (xy -2.415699 -1.260381) (xy -2.499598 -1.084459) (xy -2.570592 -0.90209) (xy -2.595842 -0.820057)
+      (xy -1.284514 -0.820057) (xy -1.284514 -1.190172) (xy -0.9144 -1.190172) (xy -0.9144 -0.820057)
+      (xy 0.892629 -0.820057) (xy 0.892629 -1.190172) (xy 1.262743 -1.190172) (xy 1.262743 -0.820057)
+      (xy 0.892629 -0.820057) (xy -0.9144 -0.820057) (xy -1.284514 -0.820057) (xy -2.595842 -0.820057)
+      (xy -2.628785 -0.713035) (xy -2.674283 -0.517054) (xy -2.70456 -0.333829) (xy -2.710207 -0.280043)
+      (xy -2.714439 -0.214741) (xy -2.717273 -0.14085) (xy -2.717988 -0.1016) (xy -0.9144 -0.1016)
+      (xy -0.9144 -0.471714) (xy -0.544286 -0.471714) (xy -0.544286 -0.1016) (xy -0.195943 -0.1016)
+      (xy -0.195943 -0.471714) (xy 0.174172 -0.471714) (xy 0.174172 -0.1016) (xy 0.544286 -0.1016)
+      (xy 0.544286 -0.471714) (xy 0.892629 -0.471714) (xy 0.892629 -0.1016) (xy 0.544286 -0.1016)
+      (xy 0.174172 -0.1016) (xy -0.195943 -0.1016) (xy -0.544286 -0.1016) (xy -0.9144 -0.1016)
+      (xy -2.717988 -0.1016) (xy -2.718723 -0.061296) (xy -2.718805 0.020994) (xy -2.717533 0.103091)
+      (xy -2.714923 0.18207) (xy -2.71099 0.255002) (xy -2.705749 0.318961) (xy -2.700976 0.359228)
+      (xy -2.665848 0.559) (xy -2.651442 0.616857) (xy -0.544286 0.616857) (xy -0.544286 0.268514)
+      (xy -0.195943 0.268514) (xy -0.195943 0.616857) (xy 0.174172 0.616857) (xy 0.174172 0.268514)
+      (xy 0.544286 0.268514) (xy 0.544286 0.616857) (xy 0.174172 0.616857) (xy -0.195943 0.616857)
+      (xy -0.544286 0.616857) (xy -2.651442 0.616857) (xy -2.617483 0.753237) (xy -2.556061 0.941573)
+      (xy -2.481761 1.123642) (xy -2.394763 1.299078) (xy -2.360491 1.357086) (xy -0.195943 1.357086)
+      (xy -0.195943 0.986971) (xy 0.174172 0.986971) (xy 0.174172 1.357086) (xy -0.195943 1.357086)
+      (xy -2.360491 1.357086) (xy -2.295247 1.467514) (xy -2.18339 1.628584) (xy -2.059374 1.781921)
+      (xy -1.942768 1.907695) (xy -1.795838 2.046806) (xy -1.642166 2.173074) (xy -1.48172 2.286516)
+      (xy -1.314466 2.387149) (xy -1.140373 2.474988) (xy -0.959407 2.550049) (xy -0.771536 2.61235)
+      (xy -0.576728 2.661905) (xy -0.37495 2.698731) (xy -0.333828 2.70456) (xy -0.280149 2.710194)
+      (xy -0.214948 2.714416) (xy -0.141149 2.717243) (xy -0.061673 2.71869) (xy 0.020556 2.718772)
+      (xy 0.102617 2.717503)) (layer B.SilkS) (width 0.01))
+  )
+  (gr_text www.ai03.me (at 246.38 104.394) (layer B.SilkS)
+    (effects (font (size 1.5 1.5) (thickness 0.3)) (justify mirror))
+  )
+  (gr_text "For default non-ISO layout, optional split back" (at 157.1625 85.725) (layer B.SilkS)
+    (effects (font (size 1.5 1.5) (thickness 0.3)) (justify mirror))
+  )
+  (gr_text "Titan - Cut-PCB keyboard plate for Voyager\n" (at 157.1625 66.675) (layer B.SilkS)
+    (effects (font (size 1.5 1.5) (thickness 0.3)) (justify mirror))
+  )
+  (gr_text www.ai03.me (at 135.73125 108.74375) (layer F.SilkS)
+    (effects (font (size 1.5 1.5) (thickness 0.3)))
+  )
   (zone (net 1) (net_name GND) (layer F.Cu) (hatch edge 0.508)
